File: kicad/dc-bias.kicad_sch (KiCad schematic)
At the start: 0 parts

Commit message: rough draft 6x4
Parts:
- added A1: Arduino_UNO_R3, Module:Arduino_UNO_R3, symbol MCU_Module:Arduino_UNO_R3
- added J1, J2: Conn_01x10, Connector_IDC:IDC-Header_2x05_P2.54mm_Vertical, symbol Connector_Generic:Conn_01x10
Other:
- added sheet non-inverting-amplifier1 (non-inverting-amplifier.kicad_sch)
- added sheet non-inverting-amplifier10 (non-inverting-amplifier.kicad_sch)
- added sheet non-inverting-amplifier11 (non-inverting-amplifier.kicad_sch)
- added sheet non-inverting-amplifier12 (non-inverting-amplifier.kicad_sch)
- added sheet non-inverting-amplifier13 (non-inverting-amplifier.kicad_sch)
- added sheet non-inverting-amplifier14 (non-inverting-amplifier.kicad_sch)
- added sheet non-inverting-amplifier15 (non-inverting-amplifier.kicad_sch)
- added sheet non-inverting-amplifier2 (non-inverting-amplifier.kicad_sch)
- added sheet non-inverting-amplifier3 (non-inverting-amplifier.kicad_sch)
- added sheet non-inverting-amplifier4 (non-inverting-amplifier.kicad_sch)
- added sheet non-inverting-amplifier5 (non-inverting-amplifier.kicad_sch)
- added sheet non-inverting-amplifier6 (non-inverting-amplifier.kicad_sch)
- added sheet non-inverting-amplifier7 (non-inverting-amplifier.kicad_sch)
- added sheet non-inverting-amplifier8 (non-inverting-amplifier.kicad_sch)
- added sheet non-inverting-amplifier9 (non-inverting-amplifier.kicad_sch)
- note added: "WRONG ARDUINO TODO TODO"

Commit message: arduino, powersupply, dac
Parts:
- removed A1: Arduino_UNO_R3, Module:Arduino_UNO_R3, symbol MCU_Module:Arduino_UNO_R3
- added A1: Arduino R4 Minima, footprints:Arduino_Uno_R4_Minima_Shield, symbol Arduino:Arduino_Uno_R4_Minima_Shield
- added U17: (no value), footprints:VHB75W, symbol VHB75W:VHB75W-Q24-S48
- added U18, U19: DAC, footprints:adafruitDAC7578, symbol adafruit:DAC7578
Other:
- removed sheet non-inverting-amplifier
- removed sheet non-inverting-amplifier1
- removed sheet non-inverting-amplifier10
- removed sheet non-inverting-amplifier11
- removed sheet non-inverting-amplifier12
- removed sheet non-inverting-amplifier13
- removed sheet non-inverting-amplifier14
- removed sheet non-inverting-amplifier2
- removed sheet non-inverting-amplifier3
- removed sheet non-inverting-amplifier4
- removed sheet non-inverting-amplifier5
- removed sheet non-inverting-amplifier6
- removed sheet non-inverting-amplifier7
- removed sheet non-inverting-amplifier8
- removed sheet non-inverting-amplifier9
- note removed: "WRONG ARDUINO TODO TODO"
- moved on the sheet: J1, J2

Commit message: finished schematic
Parts:
- removed J1, J2: Conn_01x10, Connector_IDC:IDC-Header_2x05_P2.54mm_Vertical, symbol Connector_Generic:Conn_01x10
- removed U18, U19: DAC, footprints:adafruitDAC7578, symbol adafruit:DAC7578
- added C1, C2: 100u, Capacitor_THT:CP_Radial_D7.5mm_P2.50mm, symbol Device:C_Polarized_Small_US
- added D1, D2: LED, LED_SMD:LED_1206_3216Metric_Pad1.42x1.75mm_HandSolder, symbol Device:LED
- added J3: 24V_IN, TerminalBlock_CUI:TerminalBlock_CUI_TB007-508-02_1x02_P5.08mm_Horizontal, symbol Connector_Generic:Conn_01x02
- added R1, R2: 2k2, Resistor_SMD:R_1206_3216Metric_Pad1.30x1.75mm_HandSolder, symbol Device:R_Small_US
Connections:
- net +24V: now reaches U17.1 (+V_IN)
- net +24V: now also C1.1, J3.2 (Pin_2), R1.1
- net GND: now reaches U17.3 (CASE)
- net GND: now also A1.GND1 (GND), A1.GND2 (GND), A1.GND3 (GND), A1.GND4 (SPI_GND), U17.4 (-V_IN), U17.5 (-V_OUT), C1.2, C2.2, D1.1 (K), D2.1 (K), J3.1 (Pin_1)
- net +48V: now reaches U17.9 (+V_OUT)
- net +48V: now also C2.1, R2.1
- net +3V3: now reaches A1.3V3 (3.3V)
- net +5V: now reaches A1.5V1 (5V)
- net SCL: now reaches A1.SCL
- net SDA: now reaches A1.SDA
- new net: D1.2 (A), R1.2
- new net: D2.2 (A), R2.2
- no-connect marks 0 -> 34
Other:
- removed sheet non-inverting-amplifier15
- added sheet bias-group-1 (bias-group.kicad_sch)
- added sheet bias-group1 (bias-group.kicad_sch)
- note added: "AMPLIFIERS"
- note added: "MICROCONTROL"
- note added: "POWER"
- moved on the sheet: A1, U17
