File: kicad/non-inverting-amplifier.kicad_sch (KiCad schematic)
At the start: 3 parts, among them U1 ${SIM.PARAMS}

Commit message: rough draft 6x4
Parts:
- U1: footprint (none) -> Package_SO:SOIC-8-1EP_3.9x4.9mm_P1.27mm_EP2.95x4.9mm_Mask2.71x3.4mm_ThermalVias

Commit message: arduino, powersupply, dac
Parts:
- renumbered R2 to R31, R1 to R32, U1 to U16

Commit message: finished schematic
Parts:
- R33: renamed from R31; footprint (none) -> Resistor_SMD:R_1206_3216Metric_Pad1.30x1.75mm_HandSolder
- R34: renamed from R32; value 150k -> 82k; footprint (none) -> Resistor_SMD:R_1206_3216Metric_Pad1.30x1.75mm_HandSolder
- renumbered U16 to U20
Connections:
- net IN: now reaches U20.3 (+)
- net OUT: now reaches R34.2, U20.6
Other:
- note added: "Vout = Vin (1 + Rf/R) Rf = 82k R = 10k Gain = 9.2 Vin 0-5 V, Vout 0-46 V FEEDBACK CURRENT < 1 mA R POWER < 100 mW"
- note removed: "Vout = Vin (1 + Rf/R) Rf = 150k R = 10k Gain = 16 Vin 0-5 V, Vout 0-80 V FEEDBACK CURRENT < 1 mA R POWER < 100 mW"
